File: hardware/midicontroller/mainboard.brd (EAGLE design)
At the start: 110.2 x 74.9 mm, 48 parts, among them SW1 EC12E_SW, SW2 EC12E_SW, SW3 EC12E_SW, SW4 EC12E_SW

Commit message: First prototype board design
Routing:
- net 5SDA: track 0.00 -> 131.3 mm, vias 0 -> 2
- net 5SCL: track 0.00 -> 126.2 mm, vias 0 -> 2
- net 4SDA: track 0.00 -> 102.2 mm, vias 0 -> 1
- net 4SCL: track 0.00 -> 98.6 mm, vias 0 -> 1
- net 3SDA: track 0.00 -> 82.7 mm, vias 0 -> 1
- net 3SCL: track 0.00 -> 79.1 mm, vias 0 -> 1
- net N$15: track 22.6 -> 26.1 mm, vias 0 -> 2
- added copper zone on layer 1, net GND
- added copper zone on layer 16, net VCC
Other:
- board text added: "1"
- board text added: "2"
- board text added: "3"
- board text added: "4"
- board text added: "Teensy"
